Commit message: Fix: Wrong camera orientation

File: my_robot/urdf/my_robot.xacro (robot description, xacro)
@@ -24,16 +24,12 @@
     </inertial>
     <collision name='collision'>
-	<!--origin xyz="0 0 0" rpy=" 0 0 0"/-->
       <origin xyz="0 0 0" rpy=" 0 0 0"/>
       <geometry>
-        <!--box size=".4 .2 .1"/-->
 		<cylinder radius="0.2" length="0.3"/>
       </geometry>
     </collision>
     <visual name='chassis_visual'>
-      <!--origin xyz="0 0 0" rpy=" 0 0 0"/-->
 	  <origin xyz="0 0 0" rpy=" 0 0 0"/>
       <geometry>
-        <!--box size=".4 .2 .1"/-->
 		<cylinder radius="0.2" length="0.3"/>
       </geometry>
@@ -133,28 +129,27 @@
     </collision>
   </link>
- <link name='camera_link_optical'>
-	<pose>0 0 0 -1.5707 0 -1.5707</pose>
-    <inertial>
-      <mass value="1e-5"/>
-      <origin xyz="0 0 0" rpy=" -1.5707 0 -1.5707"/>
-      <inertia
-	  ixx="1e-6" ixy="0" ixz="0"
-	  iyy="1e-6" iyz="0"
-	  izz="1e-6"
-      />
-    </inertial>
-    <visual name='camera_link_visual'>
-      <origin xyz="0 0 0" rpy=" -1.5707 0 -1.5707"/>
-      <geometry>
+	<link name='camera_link'>
+		<inertial>
+		  <mass value="0.1"/>
+		  <origin xyz="0.05 0.05 0.05" rpy=" 0 0 0"/>
+		  <inertia
+		  ixx="1e-6" ixy="0" ixz="0"
+		  iyy="1e-6" iyz="0"
+		  izz="1e-6"
+		  />
+		</inertial>
+		<visual>
+		  <origin xyz="0 0 0" rpy=" 0 0 0"/>
+		  <geometry>
 		<box size=".05 .05 .05"/>
-      </geometry>
-    </visual>
-    <collision name='camera_link_collision'>
-      <origin xyz="0 0 0" rpy=" -1.5707 0 -1.5707"/>
-      <geometry>
-	<box size=".1 .1 .1"/>
-      </geometry>
-    </collision>
-  </link>
+		  </geometry>
+		</visual>
+		<collision>
+		  <origin xyz="0 0 0" rpy=" 0 0 0"/>
+		  <geometry>
+		<box size=".05 .05 .05"/>
+		  </geometry>
+		</collision>
+	</link>
 <!-- Joints -->
   <joint name="robot_footprint_joint" type="fixed">
@@ -185,8 +180,15 @@
     <axis xyz="0 1 0" rpy="0 0 0"/>
   </joint>
-<joint type="fixed" name="camera_optical_joint">
-    <origin xyz="0 0 0" rpy="-1.5707 0 0"/>
+<joint name="camera_optical_joint" type="fixed">
+    <origin xyz="0 0 0" rpy="-1.5707 0 -1.5707"/>
+    <parent link="camera_link"/>
     <child link="camera_link_optical"/>
+  </joint>
+<joint name="camera_joint" type="fixed">
+    <origin xyz="0 0 0" rpy="0 0 0"/>
     <parent link="chassis"/>
+    <child link="camera_link"/>
   </joint>
+  <link name="camera_link_optical">
+  </link>
 </robot>

Commit message: Feat: Map generation

File: my_robot/urdf/my_robot.xacro (robot description, xacro)
@@ -3,69 +3,69 @@
   <xacro:include filename="$(find my_robot)/urdf/my_robot.gazebo" />
   <link name="robot_footprint"></link>
-<gazebo reference="left_wheel">
-    <material>Gazebo/Red</material>
-</gazebo>
-<gazebo reference="right_wheel">
-    <material>Gazebo/Red</material>
-</gazebo>
-<gazebo reference="chassis">
-    <material>Gazebo/Black</material>
-</gazebo>
-  <link name='chassis'>
-    <pose>0 0 0.1 0 0 0</pose>
-    <inertial>
-      <mass value="15.0"/>
-      <origin xyz="0.0 0 0" rpy=" 0 0 0"/>
-      <inertia
-          ixx="0.1" ixy="0" ixz="0"
-          iyy="0.1" iyz="0"
-          izz="0.1"
-      />
-    </inertial>
-    <collision name='collision'>
-      <origin xyz="0 0 0" rpy=" 0 0 0"/>
-      <geometry>
-		<cylinder radius="0.2" length="0.3"/>
-      </geometry>
-    </collision>
-    <visual name='chassis_visual'>
-	  <origin xyz="0 0 0" rpy=" 0 0 0"/>
-      <geometry>
-		<cylinder radius="0.2" length="0.3"/>
-      </geometry>
-    </visual>
-    <collision name='back_caster_collision'>
-      <origin xyz="-0.15 0 -0.15" rpy=" 0 0 0"/>
-      <geometry>
-        <sphere radius="0.0499"/>
-      </geometry>
-    </collision>
-    <visual name='back_caster_visual'>
-      <origin xyz="-0.15 0 -0.15" rpy=" 0 0 0"/>
-      <geometry>
-        <sphere radius="0.05"/>
-      </geometry>
-    </visual>
-    <collision name='front_caster_collision'>
-      <origin xyz="0.15 0 -0.15" rpy=" 0 0 0"/>
-      <geometry>
-        <sphere radius="0.0499"/>
-      </geometry>
-    </collision>
-    <visual name='front_caster_visual'>
-      <origin xyz="0.15 0 -0.15" rpy=" 0 0 0"/>
-      <geometry>
-        <sphere radius="0.05"/>
-      </geometry>
-    </visual>
-  </link>
- <link name='left_wheel'>
+  <gazebo reference="left_wheel">
+      <material>Gazebo/Red</material>
+  </gazebo>
+  <gazebo reference="right_wheel">
+      <material>Gazebo/Red</material>
+  </gazebo>
+  <gazebo reference="chassis">
+      <material>Gazebo/Black</material>
+  </gazebo>
+    <link name='chassis'>
+      <pose>0 0 0.1 0 0 0</pose>
+      <inertial>
+        <mass value="15.0"/>
+        <origin xyz="0.0 0 0" rpy=" 0 0 0"/>
+        <inertia
+            ixx="0.1" ixy="0" ixz="0"
+            iyy="0.1" iyz="0"
+            izz="0.1"
+        />
+      </inertial>
+      <collision name='collision'>
+        <origin xyz="0 0 0" rpy=" 0 0 0"/>
+        <geometry>
+  		<cylinder radius="0.2" length="0.3"/>
+        </geometry>
+      </collision>
+      <visual name='chassis_visual'>
+  	  <origin xyz="0 0 0" rpy=" 0 0 0"/>
+        <geometry>
+  		<cylinder radius="0.2" length="0.3"/>
+        </geometry>
+      </visual>
+      <collision name='back_caster_collision'>
+        <origin xyz="-0.15 0 -0.15" rpy=" 0 0 0"/>
+        <geometry>
+          <sphere radius="0.0499"/>
+        </geometry>
+      </collision>
+      <visual name='back_caster_visual'>
+        <origin xyz="-0.15 0 -0.15" rpy=" 0 0 0"/>
+        <geometry>
+          <sphere radius="0.05"/>
+        </geometry>
+      </visual>
+      <collision name='front_caster_collision'>
+        <origin xyz="0.15 0 -0.15" rpy=" 0 0 0"/>
+        <geometry>
+          <sphere radius="0.0499"/>
+        </geometry>
+      </collision>
+      <visual name='front_caster_visual'>
+        <origin xyz="0.15 0 -0.15" rpy=" 0 0 0"/>
+        <geometry>
+          <sphere radius="0.05"/>
+        </geometry>
+      </visual>
+    </link>
+  <link name='left_wheel'>
     <inertial>
       <mass value="5.0"/>
       <origin xyz="0.0 0 0" rpy=" 0 0 0"/>
       <inertia
-          ixx="0.1" ixy="0" ixz="0"
-          iyy="0.1" iyz="0"
-          izz="0.1"
+        ixx="0.1" ixy="0" ixz="0"
+        iyy="0.1" iyz="0"
+        izz="0.1"
       />
     </inertial>
@@ -82,6 +82,6 @@
       </geometry>
     </collision>
- </link>
-<link name='right_wheel'>
+  </link>
+  <link name='right_wheel'>
     <inertial>
       <mass value="5.0"/>
@@ -105,5 +105,5 @@
       </geometry>
     </collision>
- </link>
+  </link>
   <link name='hokuyo'>
     <inertial>
@@ -111,7 +111,7 @@
       <origin xyz="0 0 0" rpy=" 0 0 0"/>
       <inertia
-	  ixx="1e-6" ixy="0" ixz="0"
-	  iyy="1e-6" iyz="0"
-	  izz="1e-6"
+    ixx="1e-6" ixy="0" ixz="0"
+    iyy="1e-6" iyz="0"
+    izz="1e-6"
       />
     </inertial>
@@ -119,5 +119,5 @@
       <origin xyz="0 0 0" rpy=" 0 0 0"/>
       <geometry>
-	<mesh filename="package://my_robot/meshes/hokuyo.dae"/>
+        <mesh filename="package://my_robot/meshes/hokuyo.dae"/>
       </geometry>
     </visual>
@@ -125,32 +125,32 @@
       <origin xyz="0 0 0" rpy=" 0 0 0"/>
       <geometry>
-	<box size=".1 .1 .1"/>
+    <box size=".1 .1 .1"/>
       </geometry>
     </collision>
   </link>
-	<link name='camera_link'>
-		<inertial>
-		  <mass value="0.1"/>
-		  <origin xyz="0.05 0.05 0.05" rpy=" 0 0 0"/>
-		  <inertia
-		  ixx="1e-6" ixy="0" ixz="0"
-		  iyy="1e-6" iyz="0"
-		  izz="1e-6"
-		  />
-		</inertial>
-		<visual>
-		  <origin xyz="0 0 0" rpy=" 0 0 0"/>
-		  <geometry>
-		<box size=".05 .05 .05"/>
-		  </geometry>
-		</visual>
-		<collision>
-		  <origin xyz="0 0 0" rpy=" 0 0 0"/>
-		  <geometry>
-		<box size=".05 .05 .05"/>
-		  </geometry>
-		</collision>
-	</link>
-<!-- Joints -->
+  <link name='camera_link'>
+  	<inertial>
+  	  <mass value="0.1"/>
+  	  <origin xyz="0.05 0.05 0.05" rpy=" 0 0 0"/>
+  	  <inertia
+  	  ixx="1e-6" ixy="0" ixz="0"
+  	  iyy="1e-6" iyz="0"
+  	  izz="1e-6"
+  	  />
+  	</inertial>
+  	<visual>
+  	  <origin xyz="0 0 0" rpy=" 0 0 0"/>
+  	  <geometry>
+  	<box size=".05 .05 .05"/>
+  	  </geometry>
+  	</visual>
+  	<collision>
+  	  <origin xyz="0 0 0" rpy=" 0 0 0"/>
+  	  <geometry>
+  	<box size=".05 .05 .05"/>
+  	  </geometry>
+  	</collision>
+  </link>
+  <!-- Joints -->
   <joint name="robot_footprint_joint" type="fixed">
     <origin xyz="0 0 0" rpy="0 0 0" />
@@ -158,5 +158,5 @@
     <child link="chassis" />
   </joint>
-   <joint type="continuous" name="left_wheel_hinge">
+  <joint type="continuous" name="left_wheel_hinge">
     <origin xyz="0 0.12 -0.1" rpy="0 0 0"/>
     <child link="left_wheel"/>
@@ -166,5 +166,5 @@
     <dynamics damping="1.0" friction="1.0"/>
   </joint>
-<joint type="continuous" name="right_wheel_hinge">
+  <joint type="continuous" name="right_wheel_hinge">
     <origin xyz="0 -0.12 -0.1" rpy="0 0 0"/>
     <child link="right_wheel"/>
@@ -174,5 +174,5 @@
     <dynamics damping="1.0" friction="1.0"/>
   </joint>
-<joint type="fixed" name="hokuyo_joint">
+  <joint type="fixed" name="hokuyo_joint">
     <origin xyz=".1 0 .17" rpy="0 0 0"/>
     <child link="hokuyo"/>
@@ -180,10 +180,10 @@
     <axis xyz="0 1 0" rpy="0 0 0"/>
   </joint>
-<joint name="camera_optical_joint" type="fixed">
+  <joint name="camera_optical_joint" type="fixed">
     <origin xyz="0 0 0" rpy="-1.5707 0 -1.5707"/>
     <parent link="camera_link"/>
     <child link="camera_link_optical"/>
   </joint>
-<joint name="camera_joint" type="fixed">
+  <joint name="camera_joint" type="fixed">
     <origin xyz="0 0 0" rpy="0 0 0"/>
     <parent link="chassis"/>
